File: box_o_alps/box_o_alps.kicad_pcb (KiCad board)
At the start: 2 copper layers, 254.3 x 82.4 mm, 69 parts, among them SW00 SW_Matias_1.00u, SW01 SW_Matias_1.00u, SW02 SW_Matias_1.00u, SW03 SW_Matias_1.00u, SW04 SW_Matias_1.00u, SW05 SW_Matias_1.00u, SW06 SW_Matias_1.00u, SW07 SW_Matias_1.00u, SW08 SW_Matias_1.00u, SW09 SW_Matias_1.00u, SW10 SW_Matias_1.00u, SW11 SW_Matias_1.00u, SW12 SW_Matias_1.00u, SW13 SW_Matias_1.00u, SW14 SW_Matias_1.00u, SW15 SW_Matias_1.00u, SW16 SW_Matias_1.00u, SW17 SW_Matias_1.00u, SW18 SW_Matias_1.00u, SW19 SW_Matias_1.00u, SW20 SW_Matias_1.00u, SW21 SW_Matias_1.00u, SW22 SW_Matias_1.00u, SW23 SW_Matias_1.00u, SW24 SW_Matias_1.00u, SW25 SW_Matias_1.00u, SW26 SW_Matias_1.00u, SW27 SW_Matias_1.00u, SW28 SW_Matias_1.00u, SW29 SW_Matias_1.00u, SW33 SW_Push, SW34 SW_Push, SW35 SW_Push, SW36 SW_Push, U00 BlackPill_STLINK

Commit message: Too lazy to comment
Parts:
- removed D00, D1, D10, D11, D12, D13, D14, D15, D16, D17, D18, D19, D2, D20, D21, D22, D23, D24, D25, D26, D27, D28, D29, D3, D4, D5, D6, D7, D8, D9, REF33, REF34, REF35, REF36: D_SOD-123, Diode_SMD:D_SOD-123
- removed SW00, SW01, SW02, SW03, SW04, SW05, SW06, SW07, SW08, SW09, SW10, SW11, SW12, SW13, SW14, SW15, SW16, SW17, SW18, SW19, SW20, SW21, SW22, SW23, SW24, SW25, SW26, SW27, SW28, SW29: SW_Matias_1.00u, Button_Switch_Keyboard:SW_Matias_1.00u
- removed SW33, SW34, SW35, SW36: SW_Push, Button_Switch_Keyboard:SW_Matias_1.50u
- added U01: alps-smd-sod-123, alps_smd:alps-1u-smd-sod123, F.Cu at (50.0, 34.8)
- added U02: alps-smd-sod-123, alps_smd:alps-1u-smd-sod123, F.Cu at (69.1, 34.8)
- added U03: alps-smd-sod-123, alps_smd:alps-1u-smd-sod123, F.Cu at (88.2, 34.8)
- added U04: alps-smd-sod-123, alps_smd:alps-1u-smd-sod123, F.Cu at (107.3, 34.8)
- added U05: alps-smd-sod-123, alps_smd:alps-1u-smd-sod123, F.Cu at (183.8, 34.9)
- added U06: alps-smd-sod-123, alps_smd:alps-1u-smd-sod123, F.Cu at (202.9, 34.9)
- added U07: alps-smd-sod-123, alps_smd:alps-1u-smd-sod123, F.Cu at (222.0, 34.9)
- added U08: alps-smd-sod-123, alps_smd:alps-1u-smd-sod123, F.Cu at (241.1, 34.9)
- added U09: alps-smd-sod-123, alps_smd:alps-1u-smd-sod123, F.Cu at (260.2, 34.9)
- added U10: alps-smd-sod-123, alps_smd:alps-1u-smd-sod123, F.Cu at (30.9, 53.9)
- added U100: BlackPill_STLINK, blackpill:BlackPill_STLINK, F.Cu at (146.1, 46.9)
- added U11: alps-smd-sod-123, alps_smd:alps-1u-smd-sod123, F.Cu at (50.0, 53.9)
- added U12: alps-smd-sod-123, alps_smd:alps-1u-smd-sod123, F.Cu at (69.1, 53.9)
- added U13: alps-smd-sod-123, alps_smd:alps-1u-smd-sod123, F.Cu at (88.2, 53.9)
- added U14: alps-smd-sod-123, alps_smd:alps-1u-smd-sod123, F.Cu at (107.3, 53.9)
- added U15: alps-smd-sod-123, alps_smd:alps-1u-smd-sod123, F.Cu at (183.8, 54.0)
- added U16: alps-smd-sod-123, alps_smd:alps-1u-smd-sod123, F.Cu at (202.9, 54.0)
- added U17: alps-smd-sod-123, alps_smd:alps-1u-smd-sod123, F.Cu at (222.0, 54.0)
- added U18: alps-smd-sod-123, alps_smd:alps-1u-smd-sod123, F.Cu at (241.1, 54.0)
- added U19: alps-smd-sod-123, alps_smd:alps-1u-smd-sod123, F.Cu at (260.2, 54.0)
- added U20: alps-smd-sod-123, alps_smd:alps-1u-smd-sod123, F.Cu at (30.9, 73.0)
- added U21: alps-smd-sod-123, alps_smd:alps-1u-smd-sod123, F.Cu at (50.0, 73.0)
- added U22: alps-smd-sod-123, alps_smd:alps-1u-smd-sod123, F.Cu at (69.1, 73.0)
- added U23: alps-smd-sod-123, alps_smd:alps-1u-smd-sod123, F.Cu at (88.2, 73.0)
- added U24: alps-smd-sod-123, alps_smd:alps-1u-smd-sod123, F.Cu at (107.3, 73.0)
- added U25: alps-smd-sod-123, alps_smd:alps-1u-smd-sod123, F.Cu at (183.8, 73.0)
- added U26: alps-smd-sod-123, alps_smd:alps-1u-smd-sod123, F.Cu at (202.9, 73.0)
- added U27: alps-smd-sod-123, alps_smd:alps-1u-smd-sod123, F.Cu at (222.0, 73.0)
- added U28: alps-smd-sod-123, alps_smd:alps-1u-smd-sod123, F.Cu at (241.1, 73.0)
- added U29: alps-smd-sod-123, alps_smd:alps-1u-smd-sod123, F.Cu at (260.2, 73.0)
- added U33: alps-smd-sod-123, alps_smd:alps-1u-smd-sod123, F.Cu at (102.5, 92.1)
- added U34: alps-smd-sod-123, alps_smd:alps-1u-smd-sod123, F.Cu at (131.2, 92.1)
- added U35: alps-smd-sod-123, alps_smd:alps-1u-smd-sod123, F.Cu at (159.8, 92.1)
- added U36: alps-smd-sod-123, alps_smd:alps-1u-smd-sod123, F.Cu at (188.5, 92.1)
- U00: value BlackPill_STLINK -> alps-smd-sod-123; footprint blackpill:BlackPill_STLINK -> alps_smd:alps-1u-smd-sod123
- moved U00 144.8 mm to (30.9, 34.8)
Routing:
- net (no net): track 193.4 -> 0.00 mm
- net Net-(U100-Pad34): track 0.00 -> 160.4 mm
- net Net-(U00-Pad2): track 0.00 -> 145.5 mm
- net Net-(U100-Pad33): track 0.00 -> 140.6 mm
- net Net-(U33-Pad1): track 0.00 -> 137.1 mm
- net Net-(U100-Pad31): track 0.00 -> 129.2 mm
- net Net-(U100-Pad32): track 0.00 -> 129.0 mm
- net Net-(U01-Pad2): track 0.00 -> 126.4 mm
- net Net-(U05-Pad1): track 0.00 -> 123.5 mm
- net Net-(U20-Pad1): track 0.00 -> 123.2 mm
- net Net-(U100-Pad22): track 0.00 -> 118.3 mm
- net Net-(U10-Pad1): track 0.00 -> 113.5 mm
- net Net-(U03-Pad2): track 0.00 -> 113.4 mm
- net Net-(U100-Pad23): track 0.00 -> 113.2 mm
- net Net-(U00-Pad1): track 0.00 -> 112.0 mm
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
Commit message: Too lazy to comment
Parts:
- moved U06 19.2 mm to (183.7, 34.8)
- moved U07 19.2 mm to (202.8, 34.8)
- moved U16 19.2 mm to (183.7, 53.9)
- moved U18 19.2 mm to (221.9, 53.9)
- moved U26 19.2 mm to (183.7, 73.0)
- moved U28 19.2 mm to (221.9, 73.0)
- moved U05 19.2 mm to (164.6, 34.8)
- moved U08 19.2 mm to (221.9, 34.8)
- moved U09 19.2 mm to (241.0, 34.8)
- moved U15 19.2 mm to (164.6, 53.9)
- moved U17 19.2 mm to (202.8, 53.9)
- moved U19 19.2 mm to (241.0, 53.9)
- moved U25 19.2 mm to (164.6, 73.0)
- moved U27 19.2 mm to (202.8, 73.0)
- moved U29 19.2 mm to (241.0, 73.0)
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Connections:
- U100 pad 1: Net-(U00-Pad2) -> unconnected-(U100-Pad1)
- U100 pad 2: Net-(U01-Pad2) -> unconnected-(U100-Pad2)
- U100 pad 3: Net-(U02-Pad2) -> unconnected-(U100-Pad3)
- U100 pad 4: Net-(U03-Pad2) -> unconnected-(U100-Pad4)
- U100 pad 5: Net-(U04-Pad2) -> Net-(U00-Pad2)
- U100 pad 6: unconnected-(U100-Pad6) -> Net-(U01-Pad2)
- U100 pad 7: unconnected-(U100-Pad7) -> Net-(U02-Pad2)
- U100 pad 8: unconnected-(U100-Pad8) -> Net-(U03-Pad2)
- U100 pad 9: unconnected-(U100-Pad9) -> Net-(U04-Pad2)
Routing:
- net Net-(U04-Pad2): track 99.6 -> 82.9 mm
- net Net-(U05-Pad2): track 105.1 -> 90.0 mm
- net Net-(U07-Pad2): track 129.0 -> 117.1 mm
- net Net-(U06-Pad2): track 129.2 -> 118.1 mm
- net Net-(U10-Pad1): track 113.5 -> 102.7 mm
- net Net-(U100-Pad22): track 118.3 -> 108.0 mm
- net Net-(U00-Pad1): track 112.0 -> 103.4 mm
- net Net-(U05-Pad1): track 123.5 -> 115.5 mm
- net Net-(U100-Pad23): track 113.2 -> 105.2 mm
- net Net-(U09-Pad2): track 160.4 -> 152.9 mm
- net Net-(U100-Pad13): track 123.2 -> 115.8 mm
- net Net-(U08-Pad2): track 140.6 -> 133.8 mm
- net Net-(U00-Pad2): track 145.5 -> 139.4 mm
- net Net-(U03-Pad2): track 113.4 -> 109.2 mm
- net Net-(U100-Pad14): track 137.1 -> 133.4 mm
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Other:
- board size 254.3 x 82.4 mm -> 233.2 x 80.4 mm
