File: box_o_alps/box_o_alps.kicad_pcb (KiCad board)
At the start: 2 copper layers, 233.2 x 80.4 mm, 35 parts, among them U00 alps-smd-sod-123, U01 alps-smd-sod-123, U02 alps-smd-sod-123, U03 alps-smd-sod-123, U04 alps-smd-sod-123, U05 alps-smd-sod-123, U06 alps-smd-sod-123, U07 alps-smd-sod-123, U08 alps-smd-sod-123, U09 alps-smd-sod-123, U10 alps-smd-sod-123, U100 BlackPill_STLINK, U11 alps-smd-sod-123, U12 alps-smd-sod-123, U13 alps-smd-sod-123, U14 alps-smd-sod-123, U15 alps-smd-sod-123, U16 alps-smd-sod-123, U17 alps-smd-sod-123, U18 alps-smd-sod-123, U19 alps-smd-sod-123, U20 alps-smd-sod-123, U21 alps-smd-sod-123, U22 alps-smd-sod-123, U23 alps-smd-sod-123, U24 alps-smd-sod-123, U25 alps-smd-sod-123, U26 alps-smd-sod-123, U27 alps-smd-sod-123, U28 alps-smd-sod-123, U29 alps-smd-sod-123, U33 alps-smd-sod-123, U34 alps-smd-sod-123, U35 alps-smd-sod-123, U36 alps-smd-sod-123

Commit message: Too lazy to comment
Connections:
- U05 pad 1: Net-(U05-Pad1) -> Net-(U00-Pad1)
- U06 pad 1: Net-(U05-Pad1) -> Net-(U00-Pad1)
- U07 pad 1: Net-(U05-Pad1) -> Net-(U00-Pad1)
- U08 pad 1: Net-(U05-Pad1) -> Net-(U00-Pad1)
- U09 pad 1: Net-(U05-Pad1) -> Net-(U00-Pad1)
- U100 pad 10: unconnected-(U100-Pad10) -> Net-(U00-Pad2)
- U100 pad 11: Net-(U00-Pad1) -> Net-(U01-Pad2)
- U100 pad 12: Net-(U10-Pad1) -> Net-(U02-Pad2)
- U100 pad 13: Net-(U100-Pad13) -> Net-(U03-Pad2)
- U100 pad 14: Net-(U100-Pad14) -> Net-(U04-Pad2)
- U100 pad 16: unconnected-(U100-Pad16) -> Net-(U00-Pad1)
- U100 pad 17: unconnected-(U100-Pad17) -> Net-(U10-Pad1)
- U100 pad 22: Net-(U100-Pad22) -> unconnected-(U100-Pad22)
- U100 pad 23: Net-(U100-Pad23) -> unconnected-(U100-Pad23)
- U100 pad 24: Net-(U05-Pad1) -> Net-(U33-Pad1)
- U100 pad 26: unconnected-(U100-Pad26) -> Net-(U20-Pad1)
- U100 pad 27: unconnected-(U100-Pad27) -> Net-(U05-Pad2)
- U100 pad 28: unconnected-(U100-Pad28) -> Net-(U06-Pad2)
- U100 pad 29: unconnected-(U100-Pad29) -> Net-(U07-Pad2)
- U100 pad 30: Net-(U05-Pad2) -> Net-(U08-Pad2)
- U100 pad 31: Net-(U06-Pad2) -> Net-(U09-Pad2)
- U100 pad 32: Net-(U07-Pad2) -> unconnected-(U100-Pad32)
- U100 pad 33: Net-(U08-Pad2) -> unconnected-(U100-Pad33)
- U100 pad 34: Net-(U09-Pad2) -> unconnected-(U100-Pad34)
- U100 pad 5: Net-(U00-Pad2) -> unconnected-(U100-Pad5)
- U100 pad 6: Net-(U01-Pad2) -> unconnected-(U100-Pad6)
- U100 pad 7: Net-(U02-Pad2) -> unconnected-(U100-Pad7)
- U100 pad 8: Net-(U03-Pad2) -> unconnected-(U100-Pad8)
- U100 pad 9: Net-(U04-Pad2) -> unconnected-(U100-Pad9)
- U15 pad 1: Net-(U100-Pad23) -> Net-(U10-Pad1)
- U16 pad 1: Net-(U100-Pad23) -> Net-(U10-Pad1)
- U17 pad 1: Net-(U100-Pad23) -> Net-(U10-Pad1)
- U18 pad 1: Net-(U100-Pad23) -> Net-(U10-Pad1)
- U19 pad 1: Net-(U100-Pad23) -> Net-(U10-Pad1)
- U20 pad 1: Net-(U100-Pad13) -> Net-(U20-Pad1)
- U21 pad 1: Net-(U100-Pad13) -> Net-(U20-Pad1)
- U22 pad 1: Net-(U100-Pad13) -> Net-(U20-Pad1)
- U23 pad 1: Net-(U100-Pad13) -> Net-(U20-Pad1)
- U24 pad 1: Net-(U100-Pad13) -> Net-(U20-Pad1)
- U25 pad 1: Net-(U100-Pad22) -> Net-(U20-Pad1)
- U26 pad 1: Net-(U100-Pad22) -> Net-(U20-Pad1)
- U27 pad 1: Net-(U100-Pad22) -> Net-(U20-Pad1)
- U28 pad 1: Net-(U100-Pad22) -> Net-(U20-Pad1)
- U29 pad 1: Net-(U100-Pad22) -> Net-(U20-Pad1)
- U33 pad 1: Net-(U100-Pad14) -> Net-(U33-Pad1)
- U34 pad 1: Net-(U100-Pad14) -> Net-(U33-Pad1)
- U35 pad 1: Net-(U100-Pad14) -> Net-(U33-Pad1)
- U36 pad 1: Net-(U100-Pad14) -> Net-(U33-Pad1)
Routing:
- net Net-(U20-Pad1): track 0.00 -> 253.4 mm, vias 0 -> 2
- net Net-(U00-Pad1): track 103.4 -> 294.6 mm
- net Net-(U10-Pad1): track 102.7 -> 264.4 mm, vias 0 -> 2
- net Net-(U33-Pad1): track 0.00 -> 136.7 mm, vias 0 -> 2
- net Net-(U100-Pad14): track 133.4 -> 0.00 mm
- net Net-(U100-Pad13): track 115.8 -> 0.00 mm
- net Net-(U05-Pad1): track 115.5 -> 0.00 mm
- net Net-(U100-Pad22): track 108.0 -> 0.00 mm
- net Net-(U100-Pad23): track 105.2 -> 0.00 mm
- net Net-(U04-Pad2): track 82.9 -> 107.7 mm
- net Net-(U00-Pad2): track 139.4 -> 157.8 mm
- net Net-(U01-Pad2): track 122.6 -> 137.8 mm
- net Net-(U02-Pad2): track 106.2 -> 119.5 mm
- net Net-(U03-Pad2): track 109.2 -> 122.2 mm
- net Net-(U08-Pad2): track 133.8 -> 143.7 mm
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