File: box_o_alps/box_o_alps.kicad_sch (KiCad schematic)
At the start: 69 parts, among them SW00 SW_Push, SW01 SW_Push, SW02 SW_Push, SW03 SW_Push, SW04 SW_Push, SW05 SW_Push, SW06 SW_Push, SW07 SW_Push, SW08 SW_Push, SW09 SW_Push, SW10 SW_Push, SW11 SW_Push, SW12 SW_Push, SW13 SW_Push, SW14 SW_Push, SW15 SW_Push, SW16 SW_Push, SW17 SW_Push, SW18 SW_Push, SW19 SW_Push, SW20 SW_Push, SW21 SW_Push, SW22 SW_Push, SW23 SW_Push, SW24 SW_Push, SW25 SW_Push, SW26 SW_Push, SW27 SW_Push, SW28 SW_Push, SW29 SW_Push, SW33 SW_Push, SW34 SW_Push, SW35 SW_Push, SW36 SW_Push, U00 BlackPill_STLINK

Commit message: Too lazy to comment
Parts:
- removed D00, D01, D02, D03, D04, D05, D06, D07, D08, D09, D10, D11, D12, D13, D14, D15, D16, D17, D18, D19, D20, D21, D22, D23, D24, D25, D26, D27, D28, D29, D33, D34, D35, D36: 1N4148, Diode_SMD:D_SOD-123, symbol Diode:1N4148
- removed SW00, SW01, SW02, SW03, SW04, SW05, SW06, SW07, SW08, SW09, SW10, SW11, SW12, SW13, SW14, SW15, SW16, SW17, SW18, SW19, SW20, SW21, SW22, SW23, SW24, SW25, SW26, SW27, SW28, SW29: SW_Push, Button_Switch_Keyboard:SW_Matias_1.00u, symbol Switch:SW_Push
- removed SW33, SW34, SW35, SW36: SW_Push, Button_Switch_Keyboard:SW_Matias_1.50u, symbol Switch:SW_Push
- added U00, U01, U02, U03, U04, U05, U06, U07, U08, U09, U10, U11, U12, U13, U14, U15, U16, U17, U18, U19, U20, U21, U22, U23, U24, U25, U26, U27, U28, U29, U33, U34, U35, U36: alps-smd-sod-123, alps_smd:alps-1u-smd-sod123, symbol alps-smd:alps-smd-sod-123
- renumbered U00 to U100
Connections:
- net at U100.1 (PB12): now also U00.2, U10.2, U20.2
- net at U100.3 (PB14): now also U02.2, U12.2, U22.2
- net at U100.33 (PA7): now also U08.2, U18.2, U28.2
- net at U100.4 (PB15): now also U03.2, U13.2, U23.2, U33.2
- net at U100.14 (PB6): now also U33.1, U34.1, U35.1, U36.1
- net at U100.5 (PA8): now also U04.2, U14.2, U24.2, U34.2
- net at U100.2 (PB13): now also U01.2, U11.2, U21.2
- net at U100.32 (PA6): now also U07.2, U17.2, U27.2
- net at U100.31 (PA5): now also U06.2, U16.2, U26.2, U36.2
- net at U100.11 (PB3): now also U00.1, U01.1, U02.1, U03.1, U04.1
- net at U100.12 (PB4): now also U10.1, U11.1, U12.1, U13.1, U14.1
- net at U100.13 (PB5): now also U20.1, U21.1, U22.1, U23.1, U24.1
- net at U100.22 (PC13): now also U25.1, U26.1, U27.1, U28.1, U29.1
- net at U100.23 (PC14): now also U15.1, U16.1, U17.1, U18.1, U19.1
- net at U100.24 (PC15): now also U05.1, U06.1, U07.1, U08.1, U09.1
- net at U100.30 (PA4): now also U05.2, U15.2, U25.2, U35.2
- net at U100.34 (PB0): now also U09.2, U19.2, U29.2

Commit message: Too lazy to comment
Connections:
- net at U03.2, U13.2, U23.2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: now also U100.8 (PA11); no longer U100.4 (PB15)
- net at U01.2, U11.2, U21.2: now also U100.6 (PA9); no longer U100.2 (PB13)
- net at U00.2, U10.2, U20.2: now also U100.5 (PA8); no longer U100.1 (PB12)
- net at U02.2, U12.2, U22.2: now also U100.7 (PA10); no longer U100.3 (PB14)
- net at U04.2, U14.2, U24.2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: now also U100.9 (PA12); no longer U100.5 (PA8)
Changed lines of the file:
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@@
-    (stroke (width 0) (type default) (color 0 0 0 0))
-  )
-  (wire (pts (xy 157.48 121.92) (xy 157.48 148.59))
     (stroke (width 0) (type default) (color 0 0 0 0))
   )
@@
     (stroke (width 0) (type default) (color 0 0 0 0))
   )
-  (wire (pts (xy 210.82 97.79) (xy 210.82 161.29))
-    (stroke (width 0) (type default) (color 0 0 0 0))
-  )
   (wire (pts (xy 205.74 119.38) (xy 220.98 119.38))
     (stroke (width 0) (type default) (color 0 0 0 0))
@@
     (stroke (width 0) (type default) (color 0 0 0 0))
   )
+  (wire (pts (xy 168.91 153.67) (xy 180.34 153.67))
+    (stroke (width 0) (type default) (color 0 0 0 0))
+  )
   (wire (pts (xy 217.17 140.97) (xy 217.17 182.88))
     (stroke (width 0) (type default) (color 0 0 0 0))
@@
     (stroke (width 0) (type default) (color 0 0 0 0))
   )
+  (wire (pts (xy 171.45 148.59) (xy 180.34 148.59))
+    (stroke (width 0) (type default) (color 0 0 0 0))
+  )
   (wire (pts (xy 242.57 123.19) (xy 242.57 143.51))
     (stroke (width 0) (type default) (color 0 0 0 0))
@@
     (stroke (width 0) (type default) (color 0 0 0 0))
   )
-  (wire (pts (xy 124.46 99.06) (xy 212.09 99.06))
+  (wire (pts (xy 124.46 99.06) (xy 167.64 99.06))
     (stroke (width 0) (type default) (color 0 0 0 0))
   )
@@
     (stroke (width 0) (type default) (color 0 0 0 0))
   )
-  (wire (pts (xy 72.39 96.52) (xy 208.28 96.52))
-    (stroke (width 0) (type default) (color 0 0 0 0))
-  )
-  (wire (pts (xy 208.28 96.52) (xy 208.28 158.75))
+  (wire (pts (xy 72.39 96.52) (xy 170.18 96.52))
     (stroke (width 0) (type default) (color 0 0 0 0))
   )
@@
     (stroke (width 0) (type default) (color 0 0 0 0))
   )
-  (wire (pts (xy 157.48 148.59) (xy 180.34 148.59))
-    (stroke (width 0) (type default) (color 0 0 0 0))
-  )
   (wire (pts (xy 158.75 138.43) (xy 180.34 138.43))
     (stroke (width 0) (type default) (color 0 0 0 0))
@@
     (stroke (width 0) (type default) (color 0 0 0 0))
   )
+  (wire (pts (xy 170.18 96.52) (xy 170.18 151.13))
+    (stroke (width 0) (type default) (color 0 0 0 0))
+  )
   (wire (pts (xy 172.72 171.45) (xy 180.34 171.45))
     (stroke (width 0) (type default) (color 0 0 0 0))
@@
     (stroke (width 0) (type default) (color 0 0 0 0))
   )
+  (wire (pts (xy 167.64 99.06) (xy 167.64 156.21))
+    (stroke (width 0) (type default) (color 0 0 0 0))
+  )
   (wire (pts (xy 62.23 168.91) (xy 88.9 168.91))
     (stroke (width 0) (type default) (color 0 0 0 0))
@@
     (stroke (width 0) (type default) (color 0 0 0 0))
   )
+  (wire (pts (xy 168.91 97.79) (xy 168.91 153.67))
+    (stroke (width 0) (type default) (color 0 0 0 0))
+  )
   (wire (pts (xy 147.32 161.29) (xy 147.32 180.34))
     (stroke (width 0) (type default) (color 0 0 0 0))
@@
     (stroke (width 0) (type default) (color 0 0 0 0))
   )
-  (wire (pts (xy 212.09 163.83) (xy 205.74 163.83))
-    (stroke (width 0) (type default) (color 0 0 0 0))
-  )
   (wire (pts (xy 267.97 162.56) (xy 267.97 181.61))
     (stroke (width 0) (type default) (color 0 0 0 0))
@@
     (stroke (width 0) (type default) (color 0 0 0 0))
   )
-  (wire (pts (xy 46.99 95.25) (xy 209.55 95.25))
+  (wire (pts (xy 46.99 95.25) (xy 171.45 95.25))
     (stroke (width 0) (type default) (color 0 0 0 0))
   )
@@
     (stroke (width 0) (type default) (color 0 0 0 0))
   )
+  (wire (pts (xy 157.48 158.75) (xy 180.34 158.75))
+    (stroke (width 0) (type default) (color 0 0 0 0))
+  )
   (wire (pts (xy 215.9 116.84) (xy 215.9 138.43))
     (stroke (width 0) (type default) (color 0 0 0 0))
@@
     (stroke (width 0) (type default) (color 0 0 0 0))
   )
+  (wire (pts (xy 171.45 95.25) (xy 171.45 148.59))
+    (stroke (width 0) (type default) (color 0 0 0 0))
+  )
   (wire (pts (xy 284.48 130.81) (xy 309.88 130.81))
     (stroke (width 0) (type default) (color 0 0 0 0))
@@
     (stroke (width 0) (type default) (color 0 0 0 0))
   )
-  (wire (pts (xy 212.09 99.06) (xy 212.09 163.83))
-    (stroke (width 0) (type default) (color 0 0 0 0))
-  )
-  (wire (pts (xy 99.06 97.79) (xy 210.82 97.79))
+  (wire (pts (xy 99.06 97.79) (xy 168.91 97.79))
+    (stroke (width 0) (type default) (color 0 0 0 0))
+  )
+  (wire (pts (xy 157.48 121.92) (xy 157.48 158.75))
     (stroke (width 0) (type default) (color 0 0 0 0))
   )
@@
     (stroke (width 0) (type default) (color 0 0 0 0))
   )
+  (wire (pts (xy 170.18 151.13) (xy 180.34 151.13))
+    (stroke (width 0) (type default) (color 0 0 0 0))
+  )
   (wire (pts (xy 342.9 123.19) (xy 342.9 143.51))
     (stroke (width 0) (type default) (color 0 0 0 0))
@@
     (stroke (width 0) (type default) (color 0 0 0 0))
   )
-  (wire (pts (xy 209.55 95.25) (xy 209.55 156.21))
-    (stroke (width 0) (type default) (color 0 0 0 0))
-  )
   (wire (pts (xy 220.98 119.38) (xy 220.98 105.41))
     (stroke (width 0) (type default) (color 0 0 0 0))
@@
     (stroke (width 0) (type default) (color 0 0 0 0))
   )
+  (wire (pts (xy 167.64 156.21) (xy 180.34 156.21))
+    (stroke (width 0) (type default) (color 0 0 0 0))
+  )

Commit message: Too lazy to comment
Connections:
- net at U00.1, U01.1, U02.1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: now also U05.1, U06.1, U07.1, U08.1, U09.1, U100.16 (PB8); no longer U100.11 (PB3)
- net at U03.2, U13.2, U23.2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: now also U100.13 (PB5); no longer U100.8 (PA11)
- net at U07.2, U17.2, U27.2: now also U100.29 (PA3); no longer U100.32 (PA6)
- net at U25.1, U26.1, U27.1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: now also U100.26 (PA0), U20.1, U21.1, U22.1, U23.1, U24.1; no longer U100.22 (PC13)
- net at U08.2, U18.2, U28.2: now also U100.30 (PA4); no longer U100.33 (PA7)
- net at U05.2, U15.2, U25.2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: now also U100.27 (PA1); no longer U100.30 (PA4)
- net at U01.2, U11.2, U21.2: now also U100.11 (PB3); no longer U100.6 (PA9)
- net at U10.1, U11.1, U12.1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: now also U100.17 (PB9), U15.1, U16.1, U17.1, U18.1, U19.1; no longer U100.12 (PB4)
- net at U00.2, U10.2, U20.2: now also U100.10 (PA15); no longer U100.5 (PA8)
- net at U09.2, U19.2, U29.2: now also U100.31 (PA5); no longer U100.34 (PB0)
- net at U02.2, U12.2, U22.2: now also U100.12 (PB4); no longer U100.7 (PA10)
- net at U06.2, U16.2, U26.2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: now also U100.28 (PA2); no longer U100.31 (PA5)
- net at U33.1, U34.1, U35.1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: now also U100.24 (PC15); no longer U100.14 (PB6)
- net at U04.2, U14.2, U24.2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: now also U100.14 (PB6); no longer U100.9 (PA12)
- now unconnected: U100.23 (PC14)
