File: yask/yask.kicad_sch (KiCad schematic)
At the start: 38 parts, among them U24 alps-smd-sod-123

Commit message: Too lazy to comment
Parts:
- JLEFT1, JRIGHT1: footprint Connector_Audio:Jack_3.5mm_CUI_SJ-3523-SMT_Horizontal -> Connector_Audio:Jack_3.5mm_PJ311_Horizontal
Changed lines of the file:
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@@
     (property "Reference" "JLEFT1" (id 0) (at 187.325 156.21 0))
     (property "Value" "AudioJack3" (id 1) (at 187.325 158.75 0))
-    (property "Footprint" "Connector_Audio:Jack_3.5mm_CUI_SJ-3523-SMT_Horizontal" (id 2) (at 189.23 165.1 0)
+    (property "Footprint" "Connector_Audio:Jack_3.5mm_PJ311_Horizontal" (id 2) (at 189.23 165.1 0)
       (effects (font (size 1.27 1.27)) hide)
     )
@@
     (property "Reference" "JRIGHT1" (id 0) (at 252.095 154.94 0))
     (property "Value" "AudioJack3" (id 1) (at 252.095 157.48 0))
-    (property "Footprint" "Connector_Audio:Jack_3.5mm_CUI_SJ-3523-SMT_Horizontal" (id 2) (at 254 163.83 0)
+    (property "Footprint" "Connector_Audio:Jack_3.5mm_PJ311_Horizontal" (id 2) (at 254 163.83 0)
       (effects (font (size 1.27 1.27)) hide)
     )
@@
   (symbol_instances
     (path "/8df41c02-e5af-4c15-9219-c46c3e62fe30"
-      (reference "JLEFT1") (unit 1) (value "AudioJack3") (footprint "Connector_Audio:Jack_3.5mm_CUI_SJ-3523-SMT_Horizontal")
+      (reference "JLEFT1") (unit 1) (value "AudioJack3") (footprint "Connector_Audio:Jack_3.5mm_PJ311_Horizontal")
     )
     (path "/bebce740-91d6-4578-8b38-391ab2394b51"
-      (reference "JRIGHT1") (unit 1) (value "AudioJack3") (footprint "Connector_Audio:Jack_3.5mm_CUI_SJ-3523-SMT_Horizontal")
+      (reference "JRIGHT1") (unit 1) (value "AudioJack3") (footprint "Connector_Audio:Jack_3.5mm_PJ311_Horizontal")
     )
     (path "/fde972f0-cc24-4991-af0e-3bcb32926a01"

Commit message: Too lazy to comment
Parts:
- removed JLEFT1, JRIGHT1: AudioJack3, Connector_Audio:Jack_3.5mm_PJ311_Horizontal, symbol Connector:AudioJack3
- added Uleft1, Uright1: PJ-320A, PJ-320A_Library:PJ-320A, symbol pj320a:PJ-320A
- renumbered UL00 to UL0, UL01 to UL1, UL02 to UL2, Ul03 to UL3, Ul04 to UL4, UR00 to UR0, UR01 to UR1, UR02 to UR2, UR03 to UR3, UR04 to UR4
Connections:
- net at MRIGHT1.12 (3V3): now also Uright1.1 (Sleeve)
- net at MRIGHT1.13 (GND): now also Uright1.3 (Ring1)
- net at MRIGHT1.7 (D6): now also Uright1.2 (Tip)
- net at UL20.1, UL21.1, UL22.1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: now also MLEFT1.9 (D8)
- net at MLEFT1.1 (D0), UL14.2, UL24.2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: no longer MLEFT1.9 (D8)
- net at MLEFT1.12 (3V3): now also Uleft1.4 (Ring2)
- net at MLEFT1.13 (GND): now also Uleft1.1 (Sleeve)
- net at MLEFT1.7 (D6): now also Uleft1.2 (Tip)

Commit message: yask
Connections:
- net at MRIGHT1.12 (3V3): now also Uright1.3 (Ring1); no longer Uright1.1 (Sleeve)
- net at MRIGHT1.13 (GND): now also Uright1.1 (Sleeve); no longer Uright1.3 (Ring1)
- net at Uleft1.3 (Ring1): now also MLEFT1.12 (3V3)
- net at Uleft1.4 (Ring2): no longer MLEFT1.12 (3V3)
Changed lines of the file:
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@@
+    (stroke (width 0) (type default) (color 0 0 0 0))
+  )
+  (wire (pts (xy 213.3092 168.3004) (xy 213.3092 168.3512))
     (stroke (width 0) (type default) (color 0 0 0 0))
   )
@@
     (stroke (width 0) (type default) (color 0 0 0 0))
   )
+  (wire (pts (xy 220.218 168.148) (xy 225.552 168.148))
+    (stroke (width 0) (type default) (color 0 0 0 0))
+  )
   (wire (pts (xy 124.46 142.24) (xy 124.46 161.29))
     (stroke (width 0) (type default) (color 0 0 0 0))
@@
     (stroke (width 0) (type default) (color 0 0 0 0))
   )
-  (wire (pts (xy 241.3 173.99) (xy 274.32 173.99))
-    (stroke (width 0) (type default) (color 0 0 0 0))
-  )
   (wire (pts (xy 72.39 96.52) (xy 166.37 96.52))
     (stroke (width 0) (type default) (color 0 0 0 0))
@@
     (stroke (width 0) (type default) (color 0 0 0 0))
   )
-  (wire (pts (xy 220.345 164.465) (xy 171.45 164.465))
+  (wire (pts (xy 220.218 164.338) (xy 171.45 164.465))
     (stroke (width 0) (type default) (color 0 0 0 0))
   )
@@
     (stroke (width 0) (type default) (color 0 0 0 0))
   )
-  (wire (pts (xy 236.22 162.56) (xy 241.3 162.56))
+  (wire (pts (xy 236.22 162.56) (xy 241.046 162.56))
     (stroke (width 0) (type default) (color 0 0 0 0))
   )
@@
     (stroke (width 0) (type default) (color 0 0 0 0))
   )
-  (wire (pts (xy 275.59 134.62) (xy 275.59 166.37))
-    (stroke (width 0) (type default) (color 0 0 0 0))
-  )
   (wire (pts (xy 267.97 187.96) (xy 290.83 187.96))
     (stroke (width 0) (type default) (color 0 0 0 0))
@@
     (stroke (width 0) (type default) (color 0 0 0 0))
   )
-  (wire (pts (xy 267.97 134.62) (xy 275.59 134.62))
-    (stroke (width 0) (type default) (color 0 0 0 0))
-  )
-  (wire (pts (xy 203.2 140.97) (xy 213.36 140.97))
-    (stroke (width 0) (type default) (color 0 0 0 0))
-  )
   (wire (pts (xy 170.18 106.68) (xy 170.18 135.89))
     (stroke (width 0) (type default) (color 0 0 0 0))
   )
+  (wire (pts (xy 225.552 140.97) (xy 203.2 140.97))
+    (stroke (width 0) (type default) (color 0 0 0 0))
+  )
   (wire (pts (xy 270.51 149.86) (xy 270.51 142.24))
     (stroke (width 0) (type default) (color 0 0 0 0))
@@
     (stroke (width 0) (type default) (color 0 0 0 0))
   )
-  (wire (pts (xy 274.32 137.16) (xy 274.32 173.99))
-    (stroke (width 0) (type default) (color 0 0 0 0))
-  )
   (wire (pts (xy 231.14 137.16) (xy 231.14 109.22))
     (stroke (width 0) (type default) (color 0 0 0 0))
@@
     (stroke (width 0) (type default) (color 0 0 0 0))
   )
+  (wire (pts (xy 241.046 173.99) (xy 276.098 173.99))
+    (stroke (width 0) (type default) (color 0 0 0 0))
+  )
   (wire (pts (xy 158.75 172.72) (xy 207.01 172.72))
     (stroke (width 0) (type default) (color 0 0 0 0))
@@
     (stroke (width 0) (type default) (color 0 0 0 0))
   )
+  (wire (pts (xy 272.796 166.37) (xy 241.046 166.37))
+    (stroke (width 0) (type default) (color 0 0 0 0))
+  )
   (wire (pts (xy 147.32 161.29) (xy 147.32 180.34))
     (stroke (width 0) (type default) (color 0 0 0 0))
@@
     (stroke (width 0) (type default) (color 0 0 0 0))
   )
+  (wire (pts (xy 203.2 138.43) (xy 227.838 138.43))
+    (stroke (width 0) (type default) (color 0 0 0 0))
+  )
   (wire (pts (xy 353.06 142.24) (xy 353.06 161.29))
     (stroke (width 0) (type default) (color 0 0 0 0))
@@
     (stroke (width 0) (type default) (color 0 0 0 0))
   )
+  (wire (pts (xy 220.218 175.768) (xy 227.838 175.768))
+    (stroke (width 0) (type default) (color 0 0 0 0))
+  )
   (wire (pts (xy 157.48 173.99) (xy 157.48 168.91))
     (stroke (width 0) (type default) (color 0 0 0 0))
@@
     (stroke (width 0) (type default) (color 0 0 0 0))
   )
-  (wire (pts (xy 220.345 172.085) (xy 213.36 172.085))
+  (wire (pts (xy 267.97 137.16) (xy 272.796 137.16))
     (stroke (width 0) (type default) (color 0 0 0 0))
   )
@@
     (stroke (width 0) (type default) (color 0 0 0 0))
   )
-  (wire (pts (xy 274.32 137.16) (xy 267.97 137.16))
-    (stroke (width 0) (type default) (color 0 0 0 0))
-  )
   (wire (pts (xy 46.99 95.25) (xy 165.1 95.25))
     (stroke (width 0) (type default) (color 0 0 0 0))
@@
     (stroke (width 0) (type default) (color 0 0 0 0))
   )
+  (wire (pts (xy 267.97 134.62) (xy 276.098 134.62))
+    (stroke (width 0) (type default) (color 0 0 0 0))
+  )
   (wire (pts (xy 368.3 168.91) (xy 391.16 168.91))
     (stroke (width 0) (type default) (color 0 0 0 0))
@@
     (stroke (width 0) (type default) (color 0 0 0 0))
   )
-  (wire (pts (xy 212.09 175.895) (xy 220.345 175.895))
+  (wire (pts (xy 225.552 168.148) (xy 225.552 140.97))
     (stroke (width 0) (type default) (color 0 0 0 0))
   )
@@
     (stroke (width 0) (type default) (color 0 0 0 0))
   )
-  (wire (pts (xy 213.36 140.97) (xy 213.36 172.085))
-    (stroke (width 0) (type default) (color 0 0 0 0))
-  )
   (wire (pts (xy 171.45 146.05) (xy 165.1 146.05))
     (stroke (width 0) (type default) (color 0 0 0 0))
@@
     (stroke (width 0) (type default) (color 0 0 0 0))
   )
+  (wire (pts (xy 227.838 138.43) (xy 227.838 175.768))
+    (stroke (width 0) (type default) (color 0 0 0 0))
+  )
   (wire (pts (xy 316.23 149.86) (xy 342.9 149.86))
     (stroke (width 0) (type default) (color 0 0 0 0))
@@
     (stroke (width 0) (type default) (color 0 0 0 0))
   )
-  (wire (pts (xy 212.09 138.43) (xy 212.09 175.895))
+  (wire (pts (xy 276.098 173.99) (xy 276.098 134.62))
     (stroke (width 0) (type default) (color 0 0 0 0))
   )
@@
     (stroke (width 0) (type default) (color 0 0 0 0))
   )
-  (wire (pts (xy 241.3 166.37) (xy 275.59 166.37))
-    (stroke (width 0) (type default) (color 0 0 0 0))
-  )
   (wire (pts (xy 203.2 148.59) (xy 208.28 148.59))
     (stroke (width 0) (type default) (color 0 0 0 0))
@@
     (stroke (width 0) (type default) (color 0 0 0 0))
   )
+  (wire (pts (xy 272.796 137.16) (xy 272.796 166.37))
+    (stroke (width 0) (type default) (color 0 0 0 0))
+  )
   (wire (pts (xy 124.46 121.92) (xy 124.46 142.24))
-    (stroke (width 0) (type default) (color 0 0 0 0))
-  )
-  (wire (pts (xy 212.09 138.43) (xy 203.2 138.43))
     (stroke (width 0) (type default) (color 0 0 0 0))
   )
@@
     (pin "1")
   )
-  (symbol (lib_id "pj320a:PJ-320A") (at 219.71 179.07 0) (unit 1)
-    (in_bom yes) (on_board yes) (fields_autoplaced)
-    (property "Reference" "Uleft1" (id 0) (at 219.71 157.48 0))
-    (property "Value" "PJ-320A" (id 1) (at 219.71 160.02 0))
-    (property "Footprint" "PJ-320A_Library:PJ-320A" (id 2) (at 219.71 179.07 0)
-      (effects (font (size 1.27 1.27)) hide)
-    )
-    (property "Datasheet" "" (id 3) (at 219.71 179.07 0)
+  (symbol (lib_id "pj320a:PJ-320A") (at 219.583 178.943 0) (unit 1)
+    (in_bom yes) (on_board yes) (fields_autoplaced)
+    (property "Reference" "Uleft1" (id 0) (at 219.583 157.353 0))
+    (property "Value" "PJ-320A" (id 1) (at 219.583 159.893 0))
+    (property "Footprint" "PJ-320A_Library:PJ-320A" (id 2) (at 219.583 178.943 0))
+    (property "Datasheet" "" (id 3) (at 219.583 178.943 0)
       (effects (font (size 1.27 1.27)) hide)
     )
@@
     (pin "4")
   )
-  (symbol (lib_id "pj320a:PJ-320A") (at 241.935 177.165 0) (mirror y) (unit 1)
+  (symbol (lib_id "pj320a:PJ-320A") (at 241.681 177.165 0) (mirror y) (unit 1)
     (in_bom yes) (on_board yes)
-    (property "Reference" "Uright1" (id 0) (at 238.76 157.48 0)
+    (property "Reference" "Uright1" (id 0) (at 238.506 157.48 0)
       (effects (font (size 1.27 1.27)) (justify right))
     )
-    (property "Value" "PJ-320A" (id 1) (at 240.03 177.8 0)
+    (property "Value" "PJ-320A" (id 1) (at 239.776 177.8 0)
       (effects (font (size 1.27 1.27)) (justify right))
     )
-    (property "Footprint" "PJ-320A_Library:PJ-320A" (id 2) (at 241.935 177.165 0)
-      (effects (font (size 1.27 1.27)) hide)
-    )
-    (property "Datasheet" "" (id 3) (at 241.935 177.165 0)
-      (effects (font (size 1.27 1.27)) hide)
-    )
+    (property "Footprint" "PJ-320A_Library:PJ-320A" (id 2) (at 241.681 177.165 0)
+      (effects (font (size 1.27 1.27)) hide)
+    )
+    (property "Datasheet" "" (id 3) (at 241.681 177.165 0)
+      (effects (font (size 1.27 1.27)) hide)
+    )
